File: kicad/easyeda/mcu_wroom.kicad_sch (KiCad schematic)
At the start: 20 parts, among them J141 TYPE-C-31-M-12, SW141 RESET, SW142 BOOT, U105 ESP32-S3-WROOM-1-N16R8, U141 AMS1117-3.3, U142 USBLC6-2SC6

Commit message: Feuille MCU v2 : ajout des tirages I2C R108 / R109 (4,7 k vers +3V3), netlist revérifiée (37 nets, 0 écart)
Parts:
- added R143, R144: 5.1k, symbol Device:R
- J141: renamed from R144; value 5.1k -> TYPE-C-31-M-12; symbol Device:R -> Connector:USB_C_Receptacle_USB2.0_16P
- R108: renamed from J141; value TYPE-C-31-M-12 -> 4.7k; symbol Connector:USB_C_Receptacle_USB2.0_16P -> Device:R
- R109: renamed from R143; value 5.1k -> 4.7k
Connections:
- net GND: now also J141.A1 (GND), J141.A12 (GND), J141.B1 (GND), J141.B12 (GND), J141.S1 (SHIELD), R143.2, R144.2; no longer J141.2, R108.A1 (GND), R108.A12 (GND), R108.B1 (GND), R108.B12 (GND), R108.S1 (SHIELD), R109.2
- net I2C_SCL: now also R109.1
- net I2C_SDA: now also R108.1
- net USB_DN: now also J141.A7 (D-), J141.B7 (D-); no longer R108.A7 (D-), R108.B7 (D-)
- net USB_DP: now also J141.A6 (D+), J141.B6 (D+); no longer R108.A6 (D+), R108.B6 (D+)
- net VBUS: now also J141.A4 (VBUS), J141.A9 (VBUS), J141.B4 (VBUS), J141.B9 (VBUS); no longer R108.A4 (VBUS), R108.A9 (VBUS), R108.B4 (VBUS), R108.B9 (VBUS)
- new net: J141.B5 (CC2), R144.1
- new net: J141.A5 (CC1), R143.1
- new net +3V3: R108.2, R109.2
Other:
- note added: "2 · RESET, BOOT, console, tirages I2C"
- note removed: "2 · RESET, BOOT, console"
- moved on the sheet: R109
Changed lines of the file:
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@@
+	)
+	(symbol
+		(lib_id "Device:R")
+		(at 86.36 118.11 180)
+		(unit 1)
+		(exclude_from_sim no)
+		(in_bom yes)
+		(on_board yes)
+		(dnp no)
+		(property "Reference" "R108"
+			(at 88.9 116.84 0)
+			(effects
+				(font
+					(size 1.27 1.27)
+				)
+				(justify left)
+			)
+		)
+		(property "Value" "4.7k"
+			(at 88.9 119.38 0)
+			(effects
+				(font
+					(size 1.27 1.27)
+				)
+				(justify left)
+			)
+		)
+		(pin "1"
+		)
+		(pin "2"
+		)
+		(instances
+			(project "TriggerFlow"
+				(path "/476d30b8-f0c5-5687-9ea7-652f83ae5ac5"
+					(reference "R108")
+					(unit 1)
+				)
+			)
+		)
+	)
+	(symbol
+		(lib_id "power:+3V3")
+		(at 86.36 111.76 0)
+		(unit 1)
+		(exclude_from_sim no)
+		(in_bom yes)
+		(on_board yes)
+		(dnp no)
+		(property "Reference" "#PWR1412"
+			(at 86.36 111.76 0)
+			(hide yes)
+			(effects
+				(font
+					(size 1.27 1.27)
+				)
+			)
+		)
+		(property "Value" "+3V3"
+			(at 86.36 107.95 0)
+			(effects
+				(font
+					(size 1.27 1.27)
+				)
+			)
+		)
+		(pin "1"
+		)
+		(instances
+			(project "TriggerFlow"
+				(path "/476d30b8-f0c5-5687-9ea7-652f83ae5ac5"
+					(reference "#PWR1412")
+					(unit 1)
+				)
+			)
+		)
+	)
+	(symbol
+		(lib_id "Device:R")
+		(at 101.6 118.11 180)
+		(unit 1)
+		(exclude_from_sim no)
+		(in_bom yes)
+		(on_board yes)
+		(dnp no)
+		(property "Reference" "R109"
+			(at 104.14 116.84 0)
+			(effects
+				(font
+					(size 1.27 1.27)
+				)
+				(justify left)
+			)
+		)
+		(property "Value" "4.7k"
+			(at 104.14 119.38 0)
+			(effects
+				(font
+					(size 1.27 1.27)
+				)
+				(justify left)
+			)
+		)
+		(pin "1"
+		)
+		(pin "2"
+		)
+		(instances
+			(project "TriggerFlow"
+				(path "/476d30b8-f0c5-5687-9ea7-652f83ae5ac5"
+					(reference "R109")
+					(unit 1)
+				)
+			)
+		)
+	)
+	(symbol
+		(lib_id "power:+3V3")
+		(at 101.6 111.76 0)
+		(unit 1)
+		(exclude_from_sim no)
+		(in_bom yes)
+		(on_board yes)
+		(dnp no)
+		(property "Reference" "#PWR1413"
+			(at 101.6 111.76 0)
+			(hide yes)
+			(effects
+				(font
+					(size 1.27 1.27)
+				)
+			)
+		)
+		(property "Value" "+3V3"
+			(at 101.6 107.95 0)
+			(effects
+				(font
+					(size 1.27 1.27)
+				)
+			)
+		)
+		(pin "1"
+		)
+		(instances
+			(project "TriggerFlow"
+				(path "/476d30b8-f0c5-5687-9ea7-652f83ae5ac5"
+					(reference "#PWR1413")
+					(unit 1)
+				)
+			)
+		)
 	)
 	(symbol
@@
 		(on_board yes)
 		(dnp no)
-		(property "Reference" "#PWR1412"
+		(property "Reference" "#PWR1414"
 			(at 260.35 53.34 90)
 			(hide yes)
@@
 			(project "TriggerFlow"
 				(path "/476d30b8-f0c5-5687-9ea7-652f83ae5ac5"
-					(reference "#PWR1412")
+					(reference "#PWR1414")
 					(unit 1)
 				)
@@
 		(on_board yes)
 		(dnp no)
-		(property "Reference" "#PWR1413"
+		(property "Reference" "#PWR1415"
 			(at 270.51 55.88 90)
 			(hide yes)
@@
 			(project "TriggerFlow"
 				(path "/476d30b8-f0c5-5687-9ea7-652f83ae5ac5"
-					(reference "#PWR1413")
+					(reference "#PWR1415")
 					(unit 1)
 				)
@@
 		(on_board yes)
 		(dnp no)
-		(property "Reference" "#PWR1414"
+		(property "Reference" "#PWR1416"
 			(at 271.78 76.2 0)
 			(hide yes)
@@
 			(project "TriggerFlow"
 				(path "/476d30b8-f0c5-5687-9ea7-652f83ae5ac5"
-					(reference "#PWR1414")
+					(reference "#PWR1416")
 					(unit 1)
 				)
@@
 		(on_board yes)
 		(dnp no)
-		(property "Reference" "#PWR1415"
+		(property "Reference" "#PWR1417"
 			(at 231.14 88.9 0)
 			(hide yes)
@@
 			(project "TriggerFlow"
 				(path "/476d30b8-f0c5-5687-9ea7-652f83ae5ac5"
-					(reference "#PWR1415")
+					(reference "#PWR1417")
 					(unit 1)
 				)
@@
 		(on_board yes)
 		(dnp no)
-		(property "Reference" "#PWR1416"
+		(property "Reference" "#PWR1418"
 			(at 223.52 88.9 0)
 			(hide yes)
@@
 			(project "TriggerFlow"
 				(path "/476d30b8-f0c5-5687-9ea7-652f83ae5ac5"
-					(reference "#PWR1416")
+					(reference "#PWR1418")
 					(unit 1)
 				)
@@
 		(pts
 			(xy 50.8 124.46) (xy 66.04 124.46)
+		)
+		(stroke
+			(width 0)
+			(type default)
+		)
+	)
+	(wire
+		(pts
+			(xy 86.36 114.3) (xy 86.36 111.76)
+		)
+		(stroke
+			(width 0)
+			(type default)
+		)
+	)
+	(wire
+		(pts
+			(xy 86.36 121.92) (xy 86.36 125.73)
+		)
+		(stroke
+			(width 0)
+			(type default)
+		)
+	)
+	(wire
+		(pts
+			(xy 101.6 114.3) (xy 101.6 111.76)
+		)
+		(stroke
+			(width 0)
+			(type default)
+		)
+	)
+	(wire
+		(pts
+			(xy 101.6 121.92) (xy 101.6 125.73)
 		)
 		(stroke
@@
 		)
 	)
+	(label "I2C_SDA"
+		(at 86.36 125.73 270)
+		(effects
+			(font
+				(size 1.27 1.27)
+			)
+			(justify left bottom)
+		)
+	)
+	(label "I2C_SCL"
+		(at 101.6 125.73 270)
+		(effects
+			(font
+				(size 1.27 1.27)
+			)
+			(justify left bottom)
+		)
+	)
 	(label "VBUS"
 		(at 251.46 48.26 0)
@@
 		)
 	)
-	(text "2 · RESET, BOOT, console"
+	(text "2 · RESET, BOOT, console, tirages I2C"
 		(exclude_from_sim no)
 		(at 33.02 63.5 0)
@@
 		)
 	)
-	(text "Notes :\n• GPIO réaffectés pour le placement (v2) : TLV_OUT_1..6 = IO4-7, IO15, IO16 ; SPI SCK / MOSI = IO17 / IO18 ; I2C SCL / SDA = IO11 / IO12 ;\n  DAC2_LDAC = IO10 ; SERVO_PWM = IO48 ; vannes 1..6 = IO2, IO1, IO47, IO21, IO14, IO13 ; SHUTTER = IO38 ; FLASH_1..4 = IO39..IO42.\n• Non connectées : IO3, IO45, IO46 (démarrage), IO35-37 (PSRAM octale), IO8 et IO9 (réserve).\n• 5V_MCU par D101 (depuis +5V) ou D141 (depuis VBUS) : programmation par l'USB sans le 12 V ; l'USB n'alimente que le module.\n• U141 AMS1117-3.3 dédié au module (pointe Wi-Fi ≈ 355 mA) ; C142 + C143 au plus près de la broche 2 du module.\n• EN : 10 k / 1 µF (Espressif) + RESET ; BOOT maintenu + RESET = mode téléchargement. Console UART0 sur TP141 / TP142.\n• USB-C : CC1 / CC2 5,1 k vers GND (périphérique) ; USBLC6-2SC6 contre les décharges ; D+ / D- courtes, même longueur, sans via."
+	(text "Notes :\n• GPIO réaffectés pour le placement (v2) : TLV_OUT_1..6 = IO4-7, IO15, IO16 ; SPI SCK / MOSI = IO17 / IO18 ; I2C SCL / SDA = IO11 / IO12 ;\n  DAC2_LDAC = IO10 ; SERVO_PWM = IO48 ; vannes 1..6 = IO2, IO1, IO47, IO21, IO14, IO13 ; SHUTTER = IO38 ; FLASH_1..4 = IO39..IO42.\n• Non connectées : IO3, IO45, IO46 (démarrage), IO35-37 (PSRAM octale), IO8 et IO9 (réserve).\n• 5V_MCU par D101 (depuis +5V) ou D141 (depuis VBUS) : programmation par l'USB sans le 12 V ; l'USB n'alimente que le module.\n• U141 AMS1117-3.3 dédié au module (pointe Wi-Fi ≈ 355 mA) ; C142 + C143 au plus près de la broche 2 du module.\n• EN : 10 k / 1 µF (Espressif) + RESET ; BOOT maintenu + RESET = mode téléchargement. Console UART0 sur TP141 / TP142.\n• R108 / R109 : tirages I2C 4,7 k vers +3V3 (inchangés depuis la v1, rail des circuits du bus).\n• USB-C : CC1 / CC2 5,1 k vers GND (périphérique) ; USBLC6-2SC6 contre les décharges ; D+ / D- courtes, même longueur, sans via."
 		(exclude_from_sim no)
 		(at 30.48 137.16 0)
